File: tod.kicad_pcb (KiCad board)
At the start: 2 copper layers, 72 x 57 mm, 68 parts, among them J1 2xMVE252, J2 MV133, J3 2xMVE252, J4 MV133, Q1 BC856B, Q2 BC817, Q3 BC856B, Q4 BC817, Q5 BC856B, Q6 BC817, Q7 BC856B, Q8 BC817, U1 PC817, U2 PC817, U3 PC817, U4 PC817

Commit message: Use specific GBU8D-DC.
GBU8M-DIO does not work - it has higher forward voltage.
Parts:
- D11, D4: value GBU8* -> GBU8D-DC

Commit message: Add capacitor's voltage.
Parts:
- C1, C3, C5, C7: value 10n -> 10n/25V
- C2, C4, C6, C8: value 22u -> 22u/25V
Changed lines of the file:
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@@
 			)
 		)
-		(property "Value" "22u"
+		(property "Value" "22u/25V"
 			(at 1 3.75 90)
 			(layer "F.Fab")
@@
 			)
 		)
-		(property "Value" "22u"
+		(property "Value" "22u/25V"
 			(at 1 3.75 90)
 			(layer "F.Fab")
@@
 			)
 		)
-		(property "Value" "22u"
+		(property "Value" "22u/25V"
 			(at 1 3.75 90)
 			(layer "F.Fab")
@@
 			)
 		)
-		(property "Value" "22u"
+		(property "Value" "22u/25V"
 			(at 1 3.75 90)
 			(layer "F.Fab")
@@
 			)
 		)
-		(property "Value" "10n"
+		(property "Value" "10n/25V"
 			(at 0 -1.68 90)
 			(layer "B.Fab")
@@
 			)
 		)
-		(property "Value" "10n"
+		(property "Value" "10n/25V"
 			(at 0 -1.68 90)
 			(layer "B.Fab")
@@
 			)
 		)
-		(property "Value" "10n"
+		(property "Value" "10n/25V"
 			(at 0 -1.68 90)
 			(layer "B.Fab")
@@
 			)
 		)
-		(property "Value" "10n"
+		(property "Value" "10n/25V"
 			(at 0 -1.68 90)
 			(layer "B.Fab")

Commit message: Use RS605 bridges.
Parts:
- D11, D4: value GBU8D-DC -> RS605
Changed lines of the file:
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@@
 			)
 		)
-		(property "Value" "GBU8D-DC"
+		(property "Value" "RS605"
 			(at 7.1 -2.5 180)
 			(layer "F.Fab")
@@
 			)
 		)
-		(property "Value" "GBU8D-DC"
+		(property "Value" "RS605"
 			(at 7.1 -2.5 180)
 			(layer "F.Fab")
